Commit message: Pick and place tested. URDF modified for better workspace

File: sr_multi_description/urdf/right_srhand_ur10_joint_limited.urdf.xacro (robot description, xacro)
@@ -6,5 +6,5 @@
         <parent link="world"/>
         <child link="ra_base_link"/>
-        <origin xyz="0.0 0.0 0.0" rpy="0.0 0.0 0.0"/>
+        <origin xyz="0.0 0.0 0.1" rpy="0.0 0.0 0.0"/>
     </joint>
     <xacro:ur10_robot prefix="ra_" joint_limited="true"/>
@@ -17,5 +17,5 @@
         <parent link="ra_ee_link"/>
         <child link="rh_forearm"/>
-        <origin xyz="0.012 0.0 0.0" rpy="${pi/2.0} ${pi} ${pi/2.0}"/>
+        <origin xyz="0.012 0.0 0.0" rpy="0 ${pi/2.0} 0"/>
     </joint>
 </robot>
